File: test-boards/devsV1/power_cleanup.sch (EAGLE design)
At the start: 18 parts, among them IC2 7805L, IC3 7905L, Q1 BD139, Q2 BD140

Commit message: reworked power cleanup for darlington
Parts:
- removed Q2: BD140, transistor-power:BD140
- added Q3: MJE3055, transistor-power:MJE3055
- Q1: value BD139 -> MJE2955; device transistor-power:BD139 -> transistor-power:MJE2955
Connections:
- net +12V: now also Q3.C; no longer Q1.C
- net -12V: now also Q1.C; no longer Q2.C
- net N$1: now also Q3.B; no longer Q1.B
- net N$2: now also Q3.E; no longer Q1.E
- net N$4: now also Q1.B; no longer Q2.B
- net N$5: now also Q1.E; no longer Q2.E
Changed lines of the file:
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@@
 <parts>
 <part name="R1" library="rcl" library_urn="urn:adsk.eagle:library:334" deviceset="R-EU_" device="0207/10" package3d_urn="urn:adsk.eagle:package:23491/2" value="100K"/>
-<part name="Q1" library="transistor-power" library_urn="urn:adsk.eagle:library:400" deviceset="BD139" device="" package3d_urn="urn:adsk.eagle:package:29483/1"/>
-<part name="Q2" library="transistor-power" library_urn="urn:adsk.eagle:library:400" deviceset="BD140" device="" package3d_urn="urn:adsk.eagle:package:29483/1"/>
 <part name="C1" library="rcl" library_urn="urn:adsk.eagle:library:334" deviceset="CPOL-EU" device="E2-5" package3d_urn="urn:adsk.eagle:package:23346/2" value="2.2 uF"/>
 <part name="P-2" library="supply1" library_urn="urn:adsk.eagle:library:371" deviceset="-12V" device=""/>
@@
 <part name="JP4" library="pinhead" library_urn="urn:adsk.eagle:library:325" deviceset="PINHD-1X3" device="" package3d_urn="urn:adsk.eagle:package:22458/2"/>
 <part name="JP5" library="pinhead" library_urn="urn:adsk.eagle:library:325" deviceset="PINHD-1X3" device="" package3d_urn="urn:adsk.eagle:package:22458/2"/>
+<part name="Q3" library="transistor-power" library_urn="urn:adsk.eagle:library:400" deviceset="MJE3055" device="" package3d_urn="urn:adsk.eagle:package:29487/2"/>
+<part name="Q1" library="transistor-power" library_urn="urn:adsk.eagle:library:400" deviceset="MJE2955" device="" package3d_urn="urn:adsk.eagle:package:29487/2"/>
 </parts>
 <sheets>
@@
 <attribute name="VALUE" x="46.99" y="83.058" size="1.778" layer="96"/>
 </instance>
-<instance part="Q1" gate="1" x="60.96" y="91.44" smashed="yes" rot="R90">
-<attribute name="NAME" x="58.42" y="96.52" size="1.778" layer="95" rot="R90"/>
-<attribute name="VALUE" x="60.96" y="96.52" size="1.778" layer="96" rot="R90"/>
-</instance>
-<instance part="Q2" gate="1" x="60.96" y="53.34" smashed="yes" rot="MR90">
-<attribute name="NAME" x="63.5" y="58.42" size="1.778" layer="95" rot="MR90"/>
-<attribute name="VALUE" x="60.96" y="58.42" size="1.778" layer="96" rot="MR90"/>
-</instance>
 <instance part="C1" gate="G$1" x="60.96" y="81.28" smashed="yes">
 <attribute name="NAME" x="62.103" y="81.7626" size="1.778" layer="95"/>
@@
 <attribute name="NAME" x="171.45" y="74.295" size="1.778" layer="95"/>
 <attribute name="VALUE" x="171.45" y="60.96" size="1.778" layer="96"/>
+</instance>
+<instance part="Q3" gate="1" x="60.96" y="91.44" smashed="yes" rot="R90">
+<attribute name="NAME" x="58.42" y="96.52" size="1.778" layer="95" rot="R90"/>
+<attribute name="VALUE" x="60.96" y="96.52" size="1.778" layer="96" rot="R90"/>
+</instance>
+<instance part="Q1" gate="1" x="60.96" y="53.34" smashed="yes" rot="MR90">
+<attribute name="NAME" x="63.5" y="58.42" size="1.778" layer="95" rot="MR90"/>
+<attribute name="VALUE" x="60.96" y="58.42" size="1.778" layer="96" rot="MR90"/>
 </instance>
 </instances>
@@
 <wire x1="45.72" y1="86.36" x2="43.18" y2="86.36" width="0.1524" layer="91"/>
 <wire x1="43.18" y1="86.36" x2="43.18" y2="93.98" width="0.1524" layer="91"/>
-<pinref part="Q1" gate="1" pin="C"/>
 <wire x1="43.18" y1="93.98" x2="43.18" y2="99.06" width="0.1524" layer="91"/>
 <wire x1="55.88" y1="93.98" x2="43.18" y2="93.98" width="0.1524" layer="91"/>
 <junction x="43.18" y="93.98"/>
+<pinref part="Q3" gate="1" pin="C"/>
 </segment>
 </net>
@@
 <wire x1="43.18" y1="48.26" x2="43.18" y2="55.88" width="0.1524" layer="91"/>
 <wire x1="55.88" y1="55.88" x2="43.18" y2="55.88" width="0.1524" layer="91"/>
-<pinref part="Q2" gate="1" pin="C"/>
 <pinref part="P-3" gate="1" pin="-12V"/>
 <wire x1="43.18" y1="45.72" x2="43.18" y2="48.26" width="0.1524" layer="91"/>
 <junction x="43.18" y="48.26"/>
+<pinref part="Q1" gate="1" pin="C"/>
 </segment>
 </net>
@@
 <pinref part="C1" gate="G$1" pin="+"/>
 <wire x1="60.96" y1="88.9" x2="60.96" y2="86.36" width="0.1524" layer="91"/>
-<pinref part="Q1" gate="1" pin="B"/>
 <pinref part="R1" gate="G$1" pin="2"/>
 <wire x1="60.96" y1="86.36" x2="60.96" y2="83.82" width="0.1524" layer="91"/>
 <wire x1="55.88" y1="86.36" x2="60.96" y2="86.36" width="0.1524" layer="91"/>
 <junction x="60.96" y="86.36"/>
+<pinref part="Q3" gate="1" pin="B"/>
 </segment>
 </net>
 <net name="N$2" class="0">
 <segment>
-<pinref part="Q1" gate="1" pin="E"/>
 <pinref part="IC2" gate="A1" pin="VI"/>
 <wire x1="66.04" y1="93.98" x2="76.2" y2="93.98" width="0.1524" layer="91"/>
@@
 <wire x1="76.2" y1="88.9" x2="76.2" y2="93.98" width="0.1524" layer="91"/>
 <junction x="76.2" y="93.98"/>
+<pinref part="Q3" gate="1" pin="E"/>
 </segment>
 </net>
 <net name="N$4" class="0">
 <segment>
-<pinref part="Q2" gate="1" pin="B"/>
 <pinref part="C4" gate="G$1" pin="-"/>
 <wire x1="60.96" y1="45.72" x2="60.96" y2="48.26" width="0.1524" layer="91"/>
@@
 <wire x1="55.88" y1="48.26" x2="60.96" y2="48.26" width="0.1524" layer="91"/>
 <junction x="60.96" y="48.26"/>
+<pinref part="Q1" gate="1" pin="B"/>
 </segment>
 </net>
@@
 <wire x1="76.2" y1="50.8" x2="76.2" y2="55.88" width="0.1524" layer="91"/>
 <junction x="76.2" y="55.88"/>
-<pinref part="Q2" gate="1" pin="E"/>
 <pinref part="IC3" gate="A1" pin="VI"/>
-</segment>
-</net>
+<pinref part="Q1" gate="1" pin="E"/>
+</segment>
+</net>
