File: test-boards/devsV1/feedback.brd (EAGLE design)
At the start: 160 x 100 mm, 86 parts, among them IC1 TL074P, IC2 7805L, IC3 7905L, IC4 TL074P, IC5 TL074P, Q1 BD139, Q2 BD140

Commit message: finished board routing
Parts:
- C10, C11, C12, C13, C14, C2, C3, C5, C6, C7, C8, C9: device rcl:C025-030X050 -> rcl:C025-025X050
- IC2: device adafruit:TO92 -> linear:TO92
- R1, R10, R11, R12, R13, R14, R15, R16, R17, R18, R19, R2, R20, R21, R22, R23, R24, R25, R26, R27, R28, R29, R3, R30, R31, R32, R33, R34, R35, R36, R37, R38, R39, R4, R40, R41, R42, R43, R44, R45, R46, R47, R48, R49, R5, R50, R6, R7, R8, R9: device resistor:0207/10 -> rcl:0207/10
- moved JP7 516.0 mm to (176.5, 43.2), turned to 90 degrees
- moved R50 502.9 mm to (172.7, 36.8), turned to 270 degrees
- moved C14 495.5 mm to (168.9, 36.8), turned to 90 degrees
- moved R48 488.1 mm to (156.2, 45.7), turned to 270 degrees
- moved R49 481.8 mm to (168.9, 27.9), turned to 270 degrees
- moved JP1 479.4 mm to (168.9, 47.0), turned to 90 degrees
- moved R46 471.4 mm to (152.4, 39.4), turned to 90 degrees
- moved R47 468.4 mm to (138.4, 36.8), turned to 180 degrees
- moved R45 467.0 mm to (163.8, 41.9)
- moved R44 449.5 mm to (149.9, 34.3), turned to 270 degrees
- moved D7 438.0 mm to (152.4, 25.4), turned to 90 degrees
- moved R43 430.5 mm to (156.2, 19.1)
- moved R42 423.7 mm to (156.2, 16.5), turned to 180 degrees
- moved R41 411.8 mm to (142.2, 15.2), turned to 180 degrees
- moved R40 406.1 mm to (144.8, 12.7)
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Connections:
- net GND: now also C4.+, IC5.12; no longer C4.-, IC5.10
- net N$23: now also IC5.13; no longer IC5.9
- net N$27: now also IC5.6; no longer IC5.2
- net N$33: now also IC5.7; no longer IC5.1
- net N$34: now also IC5.3; no longer IC5.5
- net N$35: now also IC5.2; no longer IC5.6
- net N$36: now also IC5.1; no longer IC5.7
- net N$38: now also IC5.14; no longer IC5.8
- net N$4: now also C4.-; no longer C4.+
- net N$6: now also IC5.5; no longer IC5.3
Routing:
- net -5V: track 0.00 -> 245.5 mm
- net +5V: track 0.00 -> 212.7 mm
- net SIGPRE: track 0.00 -> 135.8 mm
- net SIGPOST: track 0.00 -> 118.7 mm
- net N$13: track 0.00 -> 34.8 mm
- net SOMBRERO: track 0.00 -> 31.9 mm
- net N$23: track 0.00 -> 31.1 mm
- net N$19: track 0.00 -> 30.4 mm
- net N$30: track 0.00 -> 25.5 mm
- net N$12: track 0.00 -> 25.0 mm
- net INH: track 0.00 -> 24.4 mm
- net N$28: track 0.00 -> 22.4 mm
- net N$6: track 0.00 -> 20.1 mm
- net N$24: track 0.00 -> 18.1 mm
- net N$34: track 0.00 -> 16.5 mm
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- added copper zone on layer 1, net GND
- added copper zone on layer 16, net GND
Other:
- board size 160 x 100 mm -> 182.9 x 55.5 mm

Commit message: Removed power schema from feedback, and put to separate board
Parts:
- removed C1, C4: 2.2 uF, rcl:E2-5
- removed C2, C5: 0.33uF, rcl:C025-025X050
- removed C3, C6: 1uF, rcl:C025-025X050
- removed IC2: 7805L, linear:TO92
- removed IC3: 7905L, linear:TO92
- removed JP3: 1x2, pinhead:1X02
- removed Q1: BD139, transistor-power:TO126AV
- removed Q2: BD140, transistor-power:TO126AV
- removed R1, R2: 100K, rcl:0207/10
- JP2: value 1x2 -> (none); device pinhead:1X02 -> pinhead:1X03
- moved JP4 21.7 mm to (10.2, 28.7)
- moved JP6 21.6 mm to (10.2, 23.6), turned to 270 degrees
- moved JP7 20.5 mm to (156.2, 46.2)
- moved IC5 20.3 mm to (139.7, 29.7)
- moved R42 20.3 mm to (135.9, 15.7)
- moved R43 20.3 mm to (135.9, 18.3)
- moved R44 20.3 mm to (129.5, 33.5)
- moved R45 20.3 mm to (143.5, 41.1)
- moved R48 20.3 mm to (135.9, 45.0)
- moved C13 20.3 mm to (105.4, 34.8)
- moved C9 20.3 mm to (50.8, 36.1)
- moved D2 20.3 mm to (54.6, 37.3)
- moved D4 20.3 mm to (54.6, 23.4)
- moved R17 20.3 mm to (54.6, 20.8)
- moved R18 20.3 mm to (54.6, 18.3)
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Connections:
- net N$38 renamed HEBB
- removed net +12V: JP2.1, Q1.C, R1.1
- removed net -12V: JP3.2, Q2.C, R2.1
- removed net N$1: C1.+, Q1.B, R1.2
- removed net N$2: C2.1, IC2.3, Q1.E
- removed net N$4: C4.-, Q2.B, R2.2
- removed net N$5: C5.1, IC3.2, Q2.E
- net +5V: now also JP2.3; no longer C3.1, IC2.1
- net -5V: now also JP2.1; no longer C6.1, IC3.3
- net GND: no longer C1.-, C2.2, C3.2, C4.+, C5.2, C6.2, IC2.2, IC3.1, JP3.1
Routing:
- net N$1: track 12.8 -> 0.00 mm
- net -12V: track 10.7 -> 0.00 mm
- net +12V: track 9.94 -> 0.00 mm
- net N$4: track 9.78 -> 0.00 mm
- net N$2: track 8.78 -> 0.00 mm
- net -5V: track 245.5 -> 237.0 mm
- net N$5: track 7.09 -> 0.00 mm
- net +5V: track 212.7 -> 209.1 mm
- net TPRE: track 2.54 -> 4.23 mm
- net TPOST: track 2.54 -> 4.23 mm
- net HEBB: track 14.3 -> 15.9 mm
Other:
- board size 182.9 x 55.5 mm -> 160 x 55.5 mm

Commit message: reduced size of some boards
Parts:
- C10, C11, C12, C13, C14, C7, C8, C9: device rcl:C025-025X050 -> resistor:C050-024X044
- moved R49 68.9 mm to (81.3, 12.3), turned to 180 degrees
- moved JP1 65.5 mm to (83.3, 51.3), turned to 180 degrees
- moved R40 64.8 mm to (59.7, 10.2), turned to 180 degrees
- moved R42 62.9 mm to (73.2, 20.3), turned to 270 degrees
- moved R43 60.2 mm to (75.7, 20.3), turned to 90 degrees
- moved R45 58.8 mm to (84.7, 38.9), turned to 90 degrees
- moved JP7 55.7 mm to (100.7, 51.2), turned to 180 degrees
- moved R29 54.8 mm to (27.4, 52.6), flipped to the bottom, turned to 0 degrees
- moved D7 51.3 mm to (81.8, 34.9)
- moved R31 51.2 mm to (45.2, 44.5), turned to 270 degrees
- moved R37 50.9 mm to (75.9, 46.5), turned to 90 degrees
- moved R30 50.3 mm to (48.3, 44.5), turned to 90 degrees
- moved R23 49.9 mm to (46.2, 12.7), turned to 90 degrees
- moved R21 49.7 mm to (29.2, 4.32)
- moved D6 49.3 mm to (54.4, 39.5), turned to 0 degrees
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Connections:
- net GND: now also IC5.10, IC5.8, IC5.9
- net N$11: now also IC1.10; no longer IC1.13
- net N$12: now also IC1.9; no longer IC1.12
- net N$13: now also IC1.8; no longer IC1.14
- net N$15: now also IC4.6; no longer IC4.2
- net N$18: now also IC1.13; no longer IC1.10
- net N$19: now also IC1.14; no longer IC1.8
- net N$20: now also IC1.12; no longer IC1.9
- net N$21: now also IC4.7; no longer IC4.1
- net N$26: now also IC4.3; no longer IC4.5
- net N$28: now also IC4.1; no longer IC4.7
- net N$32: now also IC4.2; no longer IC4.6
- net N$7: now also IC4.5; no longer IC4.3
Routing:
- net SIGPRE: track 135.7 -> 88.6 mm
- net SIGPOST: track 118.7 -> 87.2 mm
- net N$12: track 25.0 -> 55.8 mm
- net N$33: track 7.40 -> 37.4 mm
- net -5V: track 237.0 -> 209.4 mm
- net N$6: track 20.1 -> 47.5 mm
- net N$20: track 12.5 -> 34.8 mm
- net N$26: track 14.0 -> 33.3 mm
- net N$34: track 16.5 -> 35.8 mm
- net N$18: track 10.2 -> 28.8 mm
- net N$23: track 31.1 -> 49.1 mm
- net N$30: track 25.5 -> 7.57 mm
- net N$7: track 14.0 -> 30.4 mm
- net +5V: track 209.1 -> 193.9 mm
- net SOMBRERO: track 31.9 -> 17.5 mm
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Other:
- board size 160 x 55.5 mm -> 106.7 x 58.1 mm

Commit message: minor changes
Parts:
- moved D3 0.40 mm to (27.6, 18.2)
Routing:
- net N$13: track 24.6 -> 25.5 mm
- net N$19: track 26.5 -> 27.1 mm
Changed lines of the file:
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@@
 <attribute name="VALUE" x="18.669" y="9.144" size="1.27" layer="27" ratio="10" rot="R90"/>
 </element>
-<element name="D3" library="BeagleBone_Blue_R3" library_urn="urn:adsk.eagle:library:5828899" package="DIODE-1N4148" package3d_urn="urn:adsk.eagle:package:5829546/1" value="1N4148" x="27.178" y="18.288" smashed="yes">
-<attribute name="NAME" x="24.638" y="19.558" size="0.4064" layer="25"/>
-<attribute name="VALUE" x="25.146" y="17.78" size="0.8128" layer="21"/>
+<element name="D3" library="BeagleBone_Blue_R3" library_urn="urn:adsk.eagle:library:5828899" package="DIODE-1N4148" package3d_urn="urn:adsk.eagle:package:5829546/1" value="1N4148" x="27.559" y="18.161" smashed="yes">
+<attribute name="NAME" x="25.019" y="19.431" size="0.4064" layer="25"/>
+<attribute name="VALUE" x="25.527" y="17.653" size="0.8128" layer="21"/>
 </element>
 <element name="R15" library="rcl" library_urn="urn:adsk.eagle:library:334" package="0207/10" package3d_urn="urn:adsk.eagle:package:23491/2" value="100K" x="18.288" y="13.081" smashed="yes" rot="R90">
@@
 <wire x1="31.75" y1="20.828" x2="29.718" y2="20.828" width="0.3" layer="1"/>
 <wire x1="26.035" y1="9.525" x2="24.13" y2="9.525" width="0.3" layer="1"/>
-<wire x1="27.94" y1="19.05" x2="27.94" y2="15.24" width="0.3" layer="1"/>
-<wire x1="27.94" y1="15.24" x2="27.94" y2="11.43" width="0.3" layer="1"/>
-<wire x1="27.94" y1="11.43" x2="26.035" y2="9.525" width="0.3" layer="1"/>
-<wire x1="29.718" y1="20.828" x2="27.94" y2="19.05" width="0.3" layer="1"/>
+<wire x1="28.575" y1="19.685" x2="28.575" y2="15.875" width="0.3" layer="1"/>
+<wire x1="28.575" y1="15.875" x2="28.575" y2="12.065" width="0.3" layer="1"/>
+<wire x1="28.575" y1="12.065" x2="26.035" y2="9.525" width="0.3" layer="1"/>
+<wire x1="29.718" y1="20.828" x2="28.575" y2="19.685" width="0.3" layer="1"/>
 <wire x1="24.13" y1="14.732" x2="27.432" y2="14.732" width="0.3" layer="1"/>
-<wire x1="27.432" y1="14.732" x2="27.94" y2="15.24" width="0.3" layer="1"/>
+<wire x1="27.432" y1="14.732" x2="28.575" y2="15.875" width="0.3" layer="1"/>
 <wire x1="31.75" y1="20.828" x2="35.56" y2="20.828" width="0.3" layer="16"/>
 </signal>
@@
 <wire x1="12.192" y1="10.16" x2="13.97" y2="10.16" width="0.3" layer="1"/>
 <wire x1="13.97" y1="10.16" x2="14.351" y2="10.16" width="0.3" layer="1"/>
-<wire x1="23.3292" y1="16.5982" x2="17.9705" y2="11.2395" width="0.3" layer="1"/>
+<wire x1="23.0752" y1="16.3442" x2="17.9705" y2="11.2395" width="0.3" layer="1"/>
 <wire x1="17.9705" y1="11.2395" x2="15.621" y2="8.89" width="0.3" layer="1"/>
 <wire x1="24.13" y1="20.828" x2="24.892" y2="20.828" width="0.3" layer="1"/>
 <wire x1="26.67" y1="19.05" x2="24.892" y2="20.828" width="0.3" layer="1"/>
-<wire x1="23.3292" y1="16.5982" x2="25.4882" y2="16.5982" width="0.3" layer="1"/>
-<wire x1="25.4882" y1="16.5982" x2="26.67" y2="17.78" width="0.3" layer="1"/>
+<wire x1="23.0752" y1="16.3442" x2="25.2342" y2="16.3442" width="0.3" layer="1"/>
+<wire x1="25.2342" y1="16.3442" x2="26.67" y2="17.78" width="0.3" layer="1"/>
 <wire x1="26.67" y1="17.78" x2="26.67" y2="19.05" width="0.3" layer="1"/>
 <wire x1="24.13" y1="4.318" x2="25.908" y2="2.54" width="0.3" layer="1"/>
@@
 <contactref element="R15" pad="2"/>
 <contactref element="D3" pad="A"/>
-<wire x1="15.621" y1="13.97" x2="18.288" y2="16.637" width="0.3" layer="1"/>
+<wire x1="18.288" y1="16.637" x2="15.621" y2="13.97" width="0.3" layer="1"/>
 <wire x1="18.288" y1="16.637" x2="18.288" y2="18.161" width="0.3" layer="1"/>
-<wire x1="23.368" y1="18.288" x2="18.415" y2="18.288" width="0.3" layer="1"/>
-<wire x1="18.288" y1="18.161" x2="18.415" y2="18.288" width="0.3" layer="1"/>
+<wire x1="23.749" y1="18.161" x2="18.288" y2="18.161" width="0.3" layer="1"/>
 </signal>
 <signal name="N$18" class="1">
@@
 <contactref element="IC1" pad="14"/>
 <wire x1="22.225" y1="47.625" x2="22.225" y2="44.831" width="0.3" layer="1"/>
-<wire x1="22.225" y1="44.831" x2="26.67" y2="40.386" width="0.3" layer="1"/>
-<wire x1="26.67" y1="40.386" x2="26.67" y2="36.83" width="0.3" layer="1"/>
-<wire x1="26.67" y1="36.83" x2="27.432" y2="36.068" width="0.3" layer="1"/>
-<wire x1="27.432" y1="36.068" x2="31.75" y2="36.068" width="0.3" layer="1"/>
+<wire x1="22.225" y1="44.831" x2="24.765" y2="44.831" width="0.3" layer="1"/>
 <wire x1="39.243" y1="33.782" x2="36.703" y2="33.782" width="0.3" layer="16"/>
 <wire x1="36.703" y1="33.782" x2="35.687" y2="34.798" width="0.3" layer="16"/>
@@
 <wire x1="33.274" y1="34.798" x2="32.004" y2="36.068" width="0.3" layer="16"/>
 <wire x1="32.004" y1="36.068" x2="31.75" y2="36.068" width="0.3" layer="16"/>
+<wire x1="31.75" y1="36.068" x2="31.115" y2="36.068" width="0.3" layer="1"/>
+<wire x1="24.765" y1="44.831" x2="29.21" y2="40.386" width="0.3" layer="1"/>
+<wire x1="29.21" y1="40.386" x2="29.21" y2="36.83" width="0.3" layer="1"/>
+<wire x1="29.21" y1="36.83" x2="29.972" y2="36.068" width="0.3" layer="1"/>
+<wire x1="29.972" y1="36.068" x2="31.75" y2="36.068" width="0.3" layer="1"/>
 </signal>
 <signal name="N$20" class="1">
@@
 <wire x1="32.385" y1="42.291" x2="32.385" y2="44.831" width="0.3" layer="16"/>
 <wire x1="31.75" y1="30.988" x2="30.48" y2="30.988" width="0.3" layer="16"/>
-<wire x1="30.48" y1="30.988" x2="29.21" y2="32.258" width="0.3" layer="16"/>
+<wire x1="29.21" y1="32.258" x2="30.48" y2="30.988" width="0.3" layer="16"/>
 <wire x1="30.861" y1="42.291" x2="32.385" y2="42.291" width="0.3" layer="16"/>
-<wire x1="29.21" y1="32.258" x2="29.21" y2="40.64" width="0.3" layer="16"/>
-<wire x1="29.21" y1="40.64" x2="30.861" y2="42.291" width="0.3" layer="16"/>
+<wire x1="30.861" y1="42.291" x2="29.21" y2="40.64" width="0.3" layer="16"/>
 <wire x1="32.512" y1="30.988" x2="31.75" y2="30.988" width="0.3" layer="1"/>
 <wire x1="34.163" y1="29.337" x2="32.512" y2="30.988" width="0.3" layer="1"/>
-<wire x1="30.988" y1="18.288" x2="33.528" y2="18.288" width="0.3" layer="1"/>
-<wire x1="33.528" y1="18.288" x2="34.1496" y2="18.9096" width="0.3" layer="1"/>
+<wire x1="31.369" y1="18.161" x2="33.401" y2="18.161" width="0.3" layer="1"/>
+<wire x1="33.401" y1="18.161" x2="34.1496" y2="18.9096" width="0.3" layer="1"/>
 <wire x1="34.1496" y1="18.9096" x2="34.1496" y2="21.4122125" width="0.3" layer="1"/>
 <wire x1="34.1496" y1="21.4122125" x2="34.163" y2="21.4256125" width="0.3" layer="1"/>
 <wire x1="34.163" y1="21.4256125" x2="34.163" y2="29.337" width="0.3" layer="1"/>
+<wire x1="29.21" y1="40.64" x2="29.21" y2="32.258" width="0.3" layer="16"/>
 </signal>
 <signal name="N$7" class="1">

Commit message: measurement device init
Parts:
- moved R29 2.54 mm to (30.0, 52.5)
- moved D4 0.76 mm to (26.5, 50.3)
- moved R7 0.52 mm to (17.9, 44.3)
- moved R45 0.38 mm to (84.7, 39.2)
- moved R11 0.28 mm to (15.0, 22.0)
- moved R30 0.13 mm to (48.1, 44.5)
Routing:
- net -5V: track 209.4 -> 204.0 mm
- net N$26: track 33.3 -> 32.1 mm
- net +5V: track 193.9 -> 193.0 mm
- net N$12: track 55.8 -> 56.6 mm
- net N$33: track 37.4 -> 38.2 mm
- net N$11: track 25.2 -> 26.0 mm
- net N$15: track 9.03 -> 9.70 mm
- net N$19: track 27.1 -> 26.5 mm
Other:
- board size 106.7 x 58.1 mm -> 107.9 x 58.1 mm
