File: test-boards/Measurement device/custom_keithly.sch (EAGLE design)
At the start: 49 parts, among them IC1 TL071D, IC2 7805L, IC3 7905L, U1 AD8220, U2 INA333, U3 INA333

Commit message: added doc for required .lbr files and basic BOM
Parts:
- removed +12V, -12V: POWER_JACK, SparkFun-Connectors:POWER_JACK
- removed AGNDU1, AGNDU2, AGNDU3, BIAS, DGND, MCU_IN, MEM1, MEM2, U1OUT, U2OUT, U3OUT: (no value), pinhead:PINHD-1X1
- removed C1, C13, C16, C2, C3, C4, C5, C6, C7, C8: 0.1uF, rcl:C-EUC3216
- removed C10, C9: 10uF, rcl:C-EUC3216
- removed C14, C15: 0.33uF, rcl:C-EUC3216
- removed D1: RED, SparkFun-LED:LED-WHITE1206
- removed D2: YELLOW, SparkFun-LED:LED-WHITE1206
- removed IC1: TL071D, linear:TL071D
- removed IC2: 7805L, linear:7805L
- removed IC3: 7905L, linear:79L05Z
- removed R1, R2, R3: 100R, rcl:R-TRIMM3296W
- removed R10, R11, R12: 30R, rcl:R-EU_R0603
- removed R13, R14: 220R, rcl:R-EU_R0603
- removed R5: 10R, rcl:R-EU_R0603
- removed R6, R7, R8, R9: 100K, rcl:R-EU_R0603
- removed U$1: PS850L_BUTTON, untitled:PS850L_BUTTON
- removed U1: AD8220, untitled:AD8220
- removed U2, U3: INA333, untitled:INA333
Connections:
- removed net +5V: C1.1, C3.1, C5.1, C7.1, C9.1, D1.C, IC1.V+, U$1.P6, U1.+VS, U2.+VS, U3.+VS
- removed net -5V: C10.1, C2.2, C4.2, C6.2, C8.1, D2.A, IC1.V-, U$1.P3, U1.-VS, U2.-VS, U3.-VS
- removed net AGND: +12V.GNDBREAK, -12V.GNDBREAK, AGNDU1.1, AGNDU2.1, AGNDU3.1, C1.2, C10.2, C2.1, C3.2, C4.1, C5.2, C6.1, C7.2, C8.2, C9.2, MEM2.1, U1.REF, U2.IN-, U2.REF, U3.IN-, U3.REF
- removed net GND: +12V.GND, -12V.GND, C13.1, C14.1, C15.2, C16.2, DGND.1, IC2.GND, IC3.GND, R13.1, R14.1, R9.2
- removed net IN+: IC1.OUT, R5.1, R7.2, U1.IN+
- removed net IN-: MEM1.1, R5.2, U1.IN-
- removed net MCU_IN: MCU_IN.1, R8.1
- removed net N$1: IC1.-IN, R6.2, R7.1
- removed net N$10: -12V.PWR, C15.1, IC3.VI
- removed net N$11: C13.2, IC2.VO, U$1.P5
- removed net N$15: C16.1, IC3.VO, U$1.P2
- removed net N$2: IC1.+IN, R8.2, R9.1
- removed net N$3: R1.A, R10.1
- removed net N$4: R11.1, R2.E
- removed net N$5: R12.1, R3.E
- removed net N$7: +12V.PWR, C14.2, IC2.VI
- removed net N$8: D1.A, R13.2
- removed net N$9: D2.C, R14.2
- removed net U1OUT: U1.VOUT, U1OUT.1, U2.IN+
- removed net U1RG1: R1.S, U1.RG2
- removed net U1RG2: R10.2, U1.RG1
- removed net U2OUT: U2.VOUT, U2OUT.1, U3.IN+
- removed net U2RG1: R11.2, U2.RG1
- removed net U2RG2: R2.S, U2.RG2
- removed net U3OUT: U3.VOUT, U3OUT.1
- removed net U3RG1: R12.2, U3.RG1
- removed net U3RG2: R3.S, U3.RG2
- removed net V+: BIAS.1, R6.1

Commit message: created part of the schematic and added some datasheets
Parts:
- added C1, C2, C3, C4, C5, C6, C7, C8, C9: 0.1u, resistor:C-EUC0603K
- added JP1, JP2: (no value), pinhead:PINHD-1X1
- added R1: 80.6, resistor:R-EU_R0805
- added R2, R3, R5, R6, R7, R8: 20K, resistor:R-EU_R0603
- added R4: 300, resistor:R-EU_R0805
- added U1: AD8227BRMZ, Analog Devices_By_element14_Batch_1:AD8227BRMZ
- added U2, U6, U7: AD820ARZ-REEL7, ADI-Phase-2:AD820ARZ-REEL7
- added U3: ADS1248IPWR, Texas Instruments_By_element14_Batch_1:ADS1248IPWR
- added U4: AD5302BRMZ-REEL7, ADI-Phase-2:AD5302BRMZ-REEL7
- added U5: LM4040A20IDBZT, Texas Instruments_By_element14_Batch_1:LM4040A20IDBZT
Connections:
- new net +5V: C1.2, C3.2, C5.2, C7.2, R4.1, U1.+VS, U2.+VS, U4.VDD, U6.+VS, U7.+VS
- new net -5V: C2.2, C4.2, C6.2, C8.2, U1.-VS, U2.-VS, U6.-VS, U7.-VS
- new net 2.048V: C9.2, R4.2, R6.2, R8.2, U4.VREFA, U4.VREFB, U5.CATHODE
- new net AGND: C1.1, C2.1, C3.1, C4.1, C5.1, C6.1, C7.1, C8.1, C9.1, U4.GND, U5.ANODE
- new net DACA: JP1.1, R5.1, U6.VOUT
- new net DACB: R7.1, U2.+IN, U7.VOUT
- new net DAC_VOUTA: U4.VOUTA, U6.+IN
- new net DAC_VOUTB: U4.VOUTB, U7.+IN
- new net IN+: U1.-IN
- new net IN-: U1.+IN
- new net N$1: R1.2, U1.RG_2
- new net N$2: R1.1, U1.RG
- new net N$3: R2.1, R3.2, U2.-IN
- new net N$5: R5.2, R6.1, U6.-IN
- new net N$7: R7.2, R8.1, U7.-IN
- new net VOUTN: R3.1, U1.REF, U2.VOUT
- new net VOUTP: R2.2, U1.VOUT

Commit message: Analog part of schematic complete
Parts:
- added C10: 47u, resistor:C-EUC0603K
- added C11, C12, C13: 0.1u, resistor:C-EUC0603K
- added C14, C18: 100n, resistor:C-EUC0603K
- added C15, C16, C19, C20: 10n, resistor:C-EUC0603K
- added R10, R12, R13, R9: 1K, resistor:R-EU_R0805
- added R11: 10R, resistor:R-EU_R0805
Connections:
- new net +3V3: C11.2, U3.DVDD
- new net GND: C11.1, U3.DGND
- new net N$11: JP2.1, R11.2, R13.1
- new net N$4: C10.2, U3.VREFOUT
- new net N$6: C10.1, U3.VREFCOM
- new net N$8: C14.1, C15.2, R9.2, U3.AIN1/IEXC
- new net N$9: C14.2, C16.1, R10.2, U3.AIN0/IEXC
- net +5V: now also C12.2, U3.AVDD
- net -5V: now also C13.2, U3.AVSS
- net AGND: now also C12.1, C13.1, C15.1, C16.2, C19.1, C20.2, R11.1, R12.1
- net IN+: now also C18.2, C20.1, R13.2
- net IN-: now also C18.1, C19.2, R12.2
- net VOUTN: now also R9.1
- net VOUTP: now also R10.1
Other:
- moved on the sheet: C1, C2, C3, C4, C5, C6, C7, C8, C9, JP1, JP2, R1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

Commit message: added unconnected controlller
Parts:
- added C25: 0.1u, resistor:C-EUC0603K
- added IC1: STM32F030F4P, micro-stm_v3:STM32F030F4P
Connections:
- net +3V3: now also IC1PWR.VDD@1
- net +5V: now also C25.2
- net AGND: now also C25.1, U3.AIN2/IEXC/GPIO2, U3.AIN3/IEXC/GPIO3, U3.AIN4/IEXC/GPIO4, U3.AIN5/IEXC/GPIO5, U3.AIN6/IEXC/GPIO6, U3.AIN7/IEXC/GPIO7
Other:
- moved on the sheet: C7, C8, JP1, JP2, R7, R8, U7

Commit message: schematic v1 finished
Parts:
- added C17, C22, C23, C34: 0.1u, resistor:C-EUC0603K
- added C21: 10n, resistor:C-EUC0603K
- added C24, C28: 100n, rcl:CPOL-EUCT3216
- added C26, C30: 10u, rcl:CPOL-EUCT3216
- added C27, C29, C32: 10n, rcl:CPOL-EUCT3216
- added C31, C33: 2.2u, rcl:CPOL-EUCT3216
- added JP3: (no value), pinhead:PINHD-1X4
- added JP4, JP5: (no value), pinhead:PINHD-1X2
- added R14, R17: 150K, resistor:R-EU_R0603
- added R15, R16: 100K, resistor:R-EU_R0603
- added U10: TPS79325DBVR, Texas Instruments_By_element14_Batch_1:TPS79325DBVR
- added U8: TPS79333DBVR, Texas Instruments_By_element14_Batch_1:TPS79333DBVR
- added U9: TPS72325DBVT, Texas Instruments_By_element14_Batch_1:TPS72325DBVT
- IC1: value STM32F030F4P -> STM32F030K6T; device micro-stm_v3:STM32F030F4P -> micro-stm_v3:STM32F030K6T
Connections:
- new net +12V: C24.+, C28.+, JP4.1, R14.1, U10.EN, U10.IN, U8.EN, U8.IN
- new net -12V: C31.-, JP5.2, R17.1, U9.EN, U9.IN
- new net ADC_CS: IC1MCU.PA2, U3.~CS
- new net BAT_NEG+: R16.2, R17.2, U3.AIN4/IEXC/GPIO4
- new net BAT_POS+: R14.2, R15.2, U3.AIN2/IEXC/GPIO2
- new net CLK: IC1MCU.PA5, U3.SCLK, U4.SCLK
- new net DAC_CS: IC1MCU.PA3, U4.SYNC*
- new net DAC_LDAC: IC1MCU.PA4, U4.LDAC*
- new net DRDY: IC1MCU.PA0-WKUP, U3.~DRDY
- new net MISO: IC1MCU.PA6, U3.DOUT/~DRDY
- new net MOSI: IC1MCU.PA7, U3.DIN, U4.DIN
- new net N$10: C27.+
- new net N$12: C29.+, U10.NR
- new net N$13: C32.+, U9.NR
- new net NRST: C22.2, IC1MCU.NRST, JP3.3
- new net RX: IC1MCU.PA10
- new net START: IC1MCU.PA1, U3.START
- new net SWCLK: IC1MCU.PA14, JP3.2
- new net SWDAT: IC1MCU.PA13, JP3.1
- new net TX: IC1MCU.PA9
- net +3V3: now also C17.2, C21.2, C23.2, C26.+, IC1MCU.VDDA, IC1PWR.VDD@2, U3.~RESET, U8.OUT
- net +5V: now also C30.+, C34.1, U10.OUT
- net -5V: now also C33.-, C34.2, U9.OUT
- net AGND: now also C28.-, C29.-, C30.-, C31.+, C32.-, C33.+, JP4.2, R15.1, U10.GND, U9.GND; no longer U3.AIN2/IEXC/GPIO2, U3.AIN4/IEXC/GPIO4
- net GND: now also C17.1, C21.1, C22.1, C23.1, C24.-, C26.-, C27.-, IC1MCU.BOOT0, IC1PWR.VSS@1, IC1PWR.VSS@2, JP3.4, JP5.1, R16.1, U3.CLK, U8.GND
Other:
- moved on the sheet: C12, C13
