File: test-boards/Measurement device/custom_keithly.brd (EAGLE design)
At the start: 160 x 100 mm, 43 parts, among them IC1 STM32F030F4P, U1 AD8227BRMZ, U2 AD820ARZ-REEL7, U3 ADS1248IPWR, U4 AD5302BRMZ-REEL7, U5 LM4040A20IDBZT, U6 AD820ARZ-REEL7, U7 AD820ARZ-REEL7

Commit message: schematic v1 finished
Parts:
- added C17, C22, C23, C34: 0.1u, resistor:C0603K
- added C21: 10n, resistor:C0603K
- added C24, C28: 100n, rcl:CT3216
- added C26, C30: 10u, rcl:CT3216
- added C27, C29, C32: 10n, rcl:CT3216
- added C31, C33: 2.2u, rcl:CT3216
- added JP3: (no value), pinhead:1X04
- added JP4, JP5: (no value), pinhead:1X02
- added R14, R17: 150K, resistor:R0603
- added R15, R16: 100K, resistor:R0603
- added U10: TPS79325DBVR, Texas Instruments_By_element14_Batch_1:SOT95P280X145-5N
- added U8: TPS79333DBVR, Texas Instruments_By_element14_Batch_1:SOT95P280X145-5N
- added U9: TPS72325DBVT, Texas Instruments_By_element14_Batch_1:SOT95P280X145-5N
- IC1: value STM32F030F4P -> STM32F030K6T; device micro-stm_v3:TSSOP20-I -> micro-stm_v3:LQFP32
Connections:
- removed net VDDA: IC1.5
- removed net VSS: IC1.15
- new net +12V: C24.+, C28.+, JP4.1, R14.1, U10.1, U10.3, U8.1, U8.3
- new net -12V: C31.-, JP5.2, R17.1, U9.2, U9.3
- new net ADC_CS: IC1.8, U3.24
- new net BAT_NEG+: R16.2, R17.2, U3.13
- new net BAT_POS+: R14.2, R15.2, U3.17
- new net CLK: IC1.11, U3.28, U4.8
- new net DAC_CS: IC1.9, U4.7
- new net DAC_LDAC: IC1.10, U4.1
- new net DRDY: IC1.6, U3.25
- new net MISO: IC1.12, U3.26
- new net MOSI: IC1.13, U3.27, U4.9
- new net N$10: C27.+
- new net N$12: C29.+, U10.4
- new net N$13: C32.+, U9.4
- new net NRST: C22.2, IC1.4, JP3.3
- new net RX: IC1.20
- new net START: IC1.7, U3.23
- new net SWCLK: IC1.24, JP3.2
- new net SWDAT: IC1.23, JP3.1
- new net TX: IC1.19
- net +3V3: now also C17.2, C21.2, C23.2, C26.+, IC1.1, IC1.17, IC1.5, U3.4, U8.5; no longer IC1.16
- net +5V: now also C30.+, C34.1, U10.5
- net -5V: now also C33.-, C34.2, U9.5
- net AGND: now also C28.-, C29.-, C30.-, C31.+, C32.-, C33.+, JP4.2, R15.1, U10.2, U9.1; no longer U3.13, U3.17
- net GND: now also C17.1, C21.1, C22.1, C23.1, C24.-, C26.-, C27.-, IC1.16, IC1.31, IC1.32, JP3.4, JP5.1, R16.1, U3.3, U8.2

Commit message: pcb layout generating initiated
Parts:
- moved R17 451.5 mm to (73.7, 3.81), turned to 180 degrees
- moved R16 444.9 mm to (67.3, 3.81)
- moved JP5 444.4 mm to (71.1, 7.62)
- moved JP4 441.4 mm to (88.9, 5.08)
- moved R15 439.3 mm to (90.6, 8.13)
- moved R14 433.1 mm to (86.2, 8.13)
- moved C34 431.6 mm to (100.3, 12.7), turned to 270 degrees
- moved C22 431.4 mm to (149.9, 58.4)
- moved C24 431.4 mm to (149.9, 47.0)
- moved C27 431.4 mm to (149.9, 34.3)
- moved C17 431.4 mm to (149.9, 96.5)
- moved C21 431.4 mm to (149.9, 91.4)
- moved C23 431.4 mm to (148.6, 53.3)
- moved C25 431.4 mm to (156.2, 124.5)
- moved C26 431.4 mm to (149.9, 40.6)
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